Commit message: Added camera and joined it to chassis in urdf

File: catkin_ws/src/my_robot/urdf/my_robot.xacro (robot description, xacro)
@@ -112,5 +112,5 @@
     </collision>
   </link>
-	<!--Joints to chassis-->
+  <!--Joints to chassis-->
 	<joint type="continuous" name="left_wheel_hinge">
 	  <origin xyz="0 -0.15 0" rpy="0 0 0"/>
@@ -129,3 +129,34 @@
 	  <dynamics damping="1.0" friction="1.0"/>
 	</joint>
+  <!--Front Camera-->
+  <link name="camera">
+  	<inertial>
+      <mass value="0.1"/>
+      <origin xyz="0.0 0 0" rpy=" 0 0 0"/>
+      <inertia
+          ixx="1e-6" ixy="0" ixz="0"
+          iyy="1e-6" iyz="0"
+          izz="1e-6"
+      />
+    </inertial>
+    <collision name='camera_collision'>
+      <origin xyz="0 0 0" rpy=" 0 0 0"/>
+      <geometry>
+  		<box size=".05 .05 .05"/>
+  	  </geometry>
+    </collision>
+    <visual name='camera_visual'>
+      <origin xyz="0 0 0" rpy=" 0 0 0"/>
+      <geometry>
+  		<box size=".05 .05 .05"/>
+  	  </geometry>
+    </visual>
+  </link>
+  <!--Camera Joint-->
+  <joint name="camera_joint" type="fixed">
+  	<origin xyz="0.2 0 0" rpy="0 0 0" />
+  	<parent link="chassis" />
+  	<child link="camera" />
+  	<axis xyz="0 1 0" rpy="0 0 0" />
+  </joint>
 </robot>

Commit message: Added Lidar to the vehicle along with joined it to chassis

File: catkin_ws/src/my_robot/urdf/my_robot.xacro (robot description, xacro)
@@ -160,3 +160,34 @@
   	<axis xyz="0 1 0" rpy="0 0 0" />
   </joint>
+  <!--Lidar-->
+  <link name="Hokuyo_Lidar">
+  	<inertial>
+      <mass value="1e-5"/>
+      <origin xyz="0.0 0 0" rpy=" 0 0 0"/>
+      <inertia
+          ixx="1e-6" ixy="0" ixz="0"
+          iyy="1e-6" iyz="0"
+          izz="1e-6"
+      />
+    </inertial>
+    <collision name='Hokuyo_Lidar_collision'>
+      <origin xyz="0 0 0" rpy=" 0 0 0"/>
+      <geometry>
+  		<box size="0.1 0.1 0.1"/>
+  	  </geometry>
+    </collision>
+    <visual name='Hokuyo_Lidar_visual'>
+      <origin xyz="0 0 0" rpy=" 0 0 0"/>
+      <geometry>
+  		<mesh filename="package://my_robot/meshes/hokuyo.dae" />
+  	  </geometry>
+    </visual>
+  </link>
+  <!--LidarJoint-->
+  <joint name="Hokuyo_Lidar_joint" type="fixed">
+  	<origin xyz="0.15 0 0.1" rpy="0 0 0" />
+  	<parent link="chassis" />
+  	<child link="Hokuyo_Lidar" />
+  	<axis xyz="0 1 0" rpy="0 0 0" />
+  </joint>
 </robot>

Commit message: minor changes to my_robot xacro

File: catkin_ws/src/my_robot/urdf/my_robot.xacro (robot description, xacro)
@@ -1,6 +1,6 @@
 <?xml version='1.0'?>
 <robot name="my_robot" xmlns:xacro="http://www.ros.org/wiki/xacro">
-<xacro:include filename="$(find my_robot)/urdf/my_robot.gazebo" />
   <link name="robot_footprint"></link>
+  <xacro:include filename="$(find my_robot)/urdf/my_robot.gazebo" />
   <joint name="robot_footprint_joint" type="fixed">
     <origin xyz="0 0 0" rpy="0 0 0" />
@@ -8,5 +8,4 @@
     <child link="chassis" />
   </joint>
-  <!--Robot chassis-->
   <link name='chassis'>
     <pose>0 0 0.1 0 0 0</pose>
@@ -20,5 +19,5 @@
       />
     </inertial>
-    <collision name='collision'>
+    <collision name='chassis_collision'>
       <origin xyz="0 0 0" rpy=" 0 0 0"/>
       <geometry>
@@ -32,5 +31,4 @@
       </geometry>
     </visual>
-    <!--Casters-->
     <collision name='back_caster_collision'>
       <origin xyz="-0.15 0 -0.05" rpy=" 0 0 0"/>
@@ -58,35 +56,7 @@
     </visual>
   </link>
-	<!--Drive wheels-->
-  <link name="left_drive_wheel">
-  	<inertial>
-  	  <geometry>
-        <cylinder length="0.05" radius="0.1"/>
-      </geometry>
-      <mass value="5.0" />
-      <origin xyz="0.0 -0.01 0" rpy=" 0 1.5707 1.5707"/>
-      <inertia
-          ixx="0.1" ixy="0" ixz="0"
-          iyy="0.1" iyz="0"
-          izz="0.1"
-      />
-    </inertial>
-    <visual>
-      <mass value="5.0" />
-      <origin xyz="0 -0.01 0" rpy=" 0 1.5707 1.5707"/>
-      <geometry>
-        <cylinder length="0.05" radius="0.1"/>
-      </geometry>
-    </visual>
-    <collision>
-      <mass value="5.0"/>
-      <origin xyz="0 -0.01 0" rpy=" 0 1.5707 1.5707"/>
-      <geometry>
-        <cylinder length="0.05" radius="0.1"/>
-      </geometry>
-    </collision>
-  </link>
-  <link name="right_drive_wheel">
-  	<inertial>
+  <link name='left_drive_wheel'>
+    <pose>0 0 0 0 0 0</pose>
+    <inertial>
       <mass value="5.0"/>
       <origin xyz="0.0 0 0" rpy=" 0 1.5707 1.5707"/>
@@ -97,41 +67,62 @@
       />
     </inertial>
-    <visual>
+    <collision name='left_wheel_collision'>
       <origin xyz="0 0 0" rpy=" 0 1.5707 1.5707"/>
-      <mass value="5.0"/>
       <geometry>
-        <cylinder length="0.05" radius="0.1"/>
+        <cylinder radius="0.1" length="0.05"/>
+      </geometry>
+    </collision>
+    <visual name='left_wheel_visual'>
+      <origin xyz="0 0 0" rpy=" 0 1.5707 1.5707"/>
+      <geometry>
+        <cylinder radius="0.1" length="0.05"/>
       </geometry>
     </visual>
-    <collision>
+  </link>
+  <link name='right_drive_wheel'>
+    <pose>0 0 0 0 0 0</pose>
+    <inertial>
+      <mass value="5.0"/>
+      <origin xyz="0.0 0 0" rpy=" 0 1.5707 1.5707"/>
+      <inertia
+          ixx="0.1" ixy="0" ixz="0"
+          iyy="0.1" iyz="0"
+          izz="0.1"
+      />
+    </inertial>
+    <collision name='right_wheel_collision'>
       <origin xyz="0 0 0" rpy=" 0 1.5707 1.5707"/>
-      <mass value="5.0"/>
       <geometry>
-        <cylinder length="0.05" radius="0.1"/>
+        <cylinder radius="0.1" length="0.05"/>
       </geometry>
     </collision>
+    <visual name='right_wheel_visual'>
+      <origin xyz="0 0 0" rpy=" 0 1.5707 1.5707"/>
+      <geometry>
+        <cylinder radius="0.1" length="0.05"/>
+      </geometry>
+    </visual>
   </link>
-  <!--Joints to chassis-->
-	<joint type="continuous" name="left_wheel_hinge">
-	  <origin xyz="0 -0.15 0" rpy="0 0 0"/>
-	  <child link="left_drive_wheel"/>
-	  <parent link="chassis"/>
-	  <axis xyz="0 1 0" rpy="0 0 0"/>
-	  <limit effort="10000" velocity="1000"/>
-	  <dynamics damping="1.0" friction="1.0"/>
-	</joint>
-	<joint type="continuous" name="right_wheel_hinge">
-	  <origin xyz="0 0.15 0" rpy="0 0 0"/>
-	  <child link="right_drive_wheel"/>
-	  <parent link="chassis"/>
-	  <axis xyz="0 1 0" rpy="0 0 0"/>
-	  <limit effort="10000" velocity="1000"/>
-	  <dynamics damping="1.0" friction="1.0"/>
-	</joint>
-  <!--Front Camera-->
-  <link name="camera">
-  	<inertial>
+  <joint type="continuous" name="left_wheel_hinge">
+    <origin xyz="0 0.15 0" rpy="0 0 0"/>
+    <child link="left_wheel"/>
+    <parent link="chassis"/>
+    <axis xyz="0 1 0" rpy="0 0 0"/>
+    <limit effort="10000" velocity="1000"/>
+    <dynamics damping="1.0" friction="1.0"/>
+  </joint>
+  <joint type="continuous" name="right_wheel_hinge">
+    <origin xyz="0 -0.15 0" rpy="0 0 0"/>
+    <child link="right_wheel"/>
+    <parent link="chassis"/>
+    <axis xyz="0 1 0" rpy="0 0 0"/>
+    <limit effort="10000" velocity="1000"/>
+    <dynamics damping="1.0" friction="1.0"/>
+  </joint>
+  <link name='stereo_camera'>
+    <pose>0 0 0 0 0 0</pose>
+    <inertial>
       <mass value="0.1"/>
-      <origin xyz="0.0 0 0" rpy=" 0 0 0"/>
+      <origin xyz="0.0 0 0" rpy="0.0 0 0"/>
       <inertia
           ixx="1e-6" ixy="0" ixz="0"
@@ -143,26 +134,27 @@
       <origin xyz="0 0 0" rpy=" 0 0 0"/>
       <geometry>
-  		<box size=".05 .05 .05"/>
-  	  </geometry>
+        <box size="0.05 0.1 0.05"/>
+      </geometry>
     </collision>
     <visual name='camera_visual'>
-      <origin xyz="0 0 0" rpy=" 0 0 0"/>
+      <origin xyz="0 0 0" rpy="0 0 0"/>
       <geometry>
-  		<box size=".05 .05 .05"/>
-  	  </geometry>
+        <box size="0.05 0.05 0.05"/>
+      </geometry>
     </visual>
   </link>
-  <!--Camera Joint-->
-  <joint name="camera_joint" type="fixed">
-  	<origin xyz="0.2 0 0" rpy="0 0 0" />
-  	<parent link="chassis" />
-  	<child link="camera" />
-  	<axis xyz="0 1 0" rpy="0 0 0" />
+  <joint type="fixed" name="camera_joint">
+    <origin xyz="0.2 0 0" rpy="0 0 0"/>
+    <child link="stereo_camera"/>
+    <parent link="chassis"/>
+    <axis xyz="0 1 0" rpy="0 0 0"/>
+    <limit effort="10000" velocity="1000"/>
+    <dynamics damping="1.0" friction="1.0"/>
   </joint>
-  <!--Lidar-->
-  <link name="Hokuyo_Lidar">
-  	<inertial>
+  <link name='hokuyo_lidar'>
+    <pose>0 0 0 0 0 0</pose>
+    <inertial>
       <mass value="1e-5"/>
-      <origin xyz="0.0 0 0" rpy=" 0 0 0"/>
+      <origin xyz="0.0 0 0" rpy="0.0 0 0"/>
       <inertia
           ixx="1e-6" ixy="0" ixz="0"
@@ -171,23 +163,24 @@
       />
     </inertial>
-    <collision name='Hokuyo_Lidar_collision'>
+    <collision name='lidar_collision'>
       <origin xyz="0 0 0" rpy=" 0 0 0"/>
       <geometry>
-  		<box size="0.1 0.1 0.1"/>
-  	  </geometry>
+        <box size="0.1 0.1 0.1"/>
+      </geometry>
     </collision>
-    <visual name='Hokuyo_Lidar_visual'>
-      <origin xyz="0 0 0" rpy=" 0 0 0"/>
+    <visual name='lidar_visual'>
+      <origin xyz="0 0 0" rpy="0 0 0"/>
       <geometry>
-  		<mesh filename="package://my_robot/meshes/hokuyo.dae" />
-  	  </geometry>
+        <mesh filename="package://my_robot/meshes/hokuyo.dae"/>
+      </geometry>
     </visual>
   </link>
-  <!--LidarJoint-->
-  <joint name="Hokuyo_Lidar_joint" type="fixed">
-  	<origin xyz="0.15 0 0.1" rpy="0 0 0" />
-  	<parent link="chassis" />
-  	<child link="Hokuyo_Lidar" />
-  	<axis xyz="0 1 0" rpy="0 0 0" />
+  <joint type="fixed" name="lidar_joint">
+    <origin xyz="0.15 0.0 0.1" rpy="0 0 0"/>
+    <child link="hokuyo_lidar"/>
+    <parent link="chassis"/>
+    <axis xyz="0 1 0" rpy="0 0 0"/>
+    <limit effort="10000" velocity="1000"/>
+    <dynamics damping="1.0" friction="1.0"/>
   </joint>
 </robot>

Commit message: Modified my_robot.xacro, fixed issue with robot wheels rotating around wrong axis, fixed sensor links, fixed issue with map

File: catkin_ws/src/my_robot/urdf/my_robot.xacro (robot description, xacro)
@@ -1,6 +1,6 @@
 <?xml version='1.0'?>
 <robot name="my_robot" xmlns:xacro="http://www.ros.org/wiki/xacro">
+<xacro:include filename="$(find my_robot)/urdf/my_robot.gazebo"/>
   <link name="robot_footprint"></link>
-  <xacro:include filename="$(find my_robot)/urdf/my_robot.gazebo" />
   <joint name="robot_footprint_joint" type="fixed">
     <origin xyz="0 0 0" rpy="0 0 0" />
@@ -8,8 +8,9 @@
     <child link="chassis" />
   </joint>
+  <!--Robot chassis-->
   <link name='chassis'>
     <pose>0 0 0.1 0 0 0</pose>
     <inertial>
-      <mass value="15.0"/>
+      <mass value="25.0"/>
       <origin xyz="0.0 0 0" rpy=" 0 0 0"/>
       <inertia
@@ -19,8 +20,8 @@
       />
     </inertial>
-    <collision name='chassis_collision'>
-      <origin xyz="0 0 0" rpy=" 0 0 0"/>
-      <geometry>
-        <box size=".4 .2 .1"/>
+    <collision name='collision'>
+      <origin xyz="0 0 0" rpy=" 0 0 0"/>
+      <geometry>
+        <box size=".7 .5 .15"/>
       </geometry>
     </collision>
@@ -28,37 +29,65 @@
       <origin xyz="0 0 0" rpy=" 0 0 0"/>
       <geometry>
-        <box size=".4 .2 .1"/>
-      </geometry>
-    </visual>
-    <collision name='back_caster_collision'>
-      <origin xyz="-0.15 0 -0.05" rpy=" 0 0 0"/>
-      <geometry>
-        <sphere radius="0.0499"/>
-      </geometry>
-    </collision>
-    <visual name='back_caster_visual'>
-      <origin xyz="-0.15 0 -0.05" rpy=" 0 0 0"/>
-      <geometry>
-        <sphere radius="0.05"/>
-      </geometry>
-    </visual>
-    <collision name='front_caster_collision'>
-      <origin xyz="0.15 0 -0.05" rpy=" 0 0 0"/>
-      <geometry>
-        <sphere radius="0.0499"/>
-      </geometry>
-    </collision>
-    <visual name='front_caster_visual'>
-      <origin xyz="0.15 0 -0.05" rpy=" 0 0 0"/>
-      <geometry>
-        <sphere radius="0.05"/>
-      </geometry>
-    </visual>
-  </link>
-  <link name='left_drive_wheel'>
-    <pose>0 0 0 0 0 0</pose>
-    <inertial>
-      <mass value="5.0"/>
-      <origin xyz="0.0 0 0" rpy=" 0 1.5707 1.5707"/>
+        <box size=".7 .5 .15"/>
+      </geometry>
+    </visual>
+    <!--Casters-->
+    <collision name='rear_left_caster_collision'>
+      <origin xyz="-0.3 -0.2 -0.1" rpy=" 0 0 0"/>
+      <geometry>
+        <sphere radius="0.0499"/>
+      </geometry>
+    </collision>
+    <visual name='rear_left_caster_visual'>
+      <origin xyz="-0.3 -0.2 -0.1" rpy=" 0 0 0"/>
+      <geometry>
+        <sphere radius="0.05"/>
+      </geometry>
+    </visual>
+   <collision name='rear_right_caster_collision'>
+      <origin xyz="0.3 0.2 -0.1" rpy=" 0 0 0"/>
+      <geometry>
+        <sphere radius="0.0499"/>
+      </geometry>
+    </collision>
+    <visual name='rear_right_caster_visual'>
+      <origin xyz="0.3 0.2 -0.1" rpy=" 0 0 0"/>
+      <geometry>
+        <sphere radius="0.05"/>
+      </geometry>
+    </visual>
+    <collision name='front_left_caster_collision'>
+      <origin xyz="0.3 -0.2 -0.1" rpy=" 0 0 0"/>
+      <geometry>
+        <sphere radius="0.0499"/>
+      </geometry>
+    </collision>
+    <visual name='front_left_caster_visual'>
+      <origin xyz="0.3 -0.2 -0.1" rpy=" 0 0 0"/>
+      <geometry>
+        <sphere radius="0.05"/>
+      </geometry>
+    </visual>
+    <collision name='front_right_caster_collision'>
+      <origin xyz="-0.3 0.2 -0.1" rpy=" 0 0 0"/>
+      <geometry>
+        <sphere radius="0.0499"/>
+      </geometry>
+    </collision>
+    <visual name='front_right_caster_visual'>
+      <origin xyz="-0.3 0.2 -0.1" rpy=" 0 0 0"/>
+      <geometry>
+        <sphere radius="0.05"/>
+      </geometry>
+    </visual>
+  </link>
+	<!--Drive wheels-->
+  <link name="right_drive_wheel">
+  	<inertial>
+  	  <geometry>
+        <cylinder length="0.05" radius="0.1"/>
+      </geometry>
+      <mass value="5.0" />
+      <origin xyz="0.0 0 -0" rpy=" 0 1.5707 1.5707"/>
       <inertia
           ixx="0.1" ixy="0" ixz="0"
@@ -67,22 +96,23 @@
       />
     </inertial>
-    <collision name='left_wheel_collision'>
-      <origin xyz="0 0 0" rpy=" 0 1.5707 1.5707"/>
-      <geometry>
-        <cylinder radius="0.1" length="0.05"/>
-      </geometry>
-    </collision>
-    <visual name='left_wheel_visual'>
-      <origin xyz="0 0 0" rpy=" 0 1.5707 1.5707"/>
-      <geometry>
-        <cylinder radius="0.1" length="0.05"/>
-      </geometry>
-    </visual>
-  </link>
-  <link name='right_drive_wheel'>
-    <pose>0 0 0 0 0 0</pose>
-    <inertial>
-      <mass value="5.0"/>
-      <origin xyz="0.0 0 0" rpy=" 0 1.5707 1.5707"/>
+    <visual>
+      <mass value="5.0" />
+      <origin xyz="0 0 -0" rpy=" 0 1.5707 1.5707"/>
+      <geometry>
+        <cylinder length="0.05" radius="0.1"/>
+      </geometry>
+    </visual>
+    <collision>
+      <mass value="5.0"/>
+      <origin xyz="0 0 -0" rpy=" 0 1.5707 1.5707"/>
+      <geometry>
+        <cylinder length="0.05" radius="0.1"/>
+      </geometry>
+    </collision>
+  </link>
+  <link name="left_drive_wheel">
+  	<inertial>
+      <mass value="5.0"/>
+      <origin xyz="0.0 -0 -0" rpy=" 0 1.5707 1.5707"/>
       <inertia
           ixx="0.1" ixy="0" ixz="0"
@@ -91,38 +121,41 @@
       />
     </inertial>
-    <collision name='right_wheel_collision'>
+    <visual>
       <origin xyz="0 0 0" rpy=" 0 1.5707 1.5707"/>
-      <geometry>
-        <cylinder radius="0.1" length="0.05"/>
-      </geometry>
-    </collision>
-    <visual name='right_wheel_visual'>
+      <mass value="5.0"/>
+      <geometry>
+        <cylinder length="0.05" radius="0.1"/>
+      </geometry>
+    </visual>
+    <collision>
       <origin xyz="0 0 0" rpy=" 0 1.5707 1.5707"/>
-      <geometry>
-        <cylinder radius="0.1" length="0.05"/>
-      </geometry>
-    </visual>
-  </link>
-  <joint type="continuous" name="left_wheel_hinge">
-    <origin xyz="0 0.15 0" rpy="0 0 0"/>
-    <child link="left_wheel"/>
-    <parent link="chassis"/>
-    <axis xyz="0 1 0" rpy="0 0 0"/>
-    <limit effort="10000" velocity="1000"/>
-    <dynamics damping="1.0" friction="1.0"/>
-  </joint>
-  <joint type="continuous" name="right_wheel_hinge">
-    <origin xyz="0 -0.15 0" rpy="0 0 0"/>
-    <child link="right_wheel"/>
-    <parent link="chassis"/>
-    <axis xyz="0 1 0" rpy="0 0 0"/>
-    <limit effort="10000" velocity="1000"/>
-    <dynamics damping="1.0" friction="1.0"/>
-  </joint>
-  <link name='stereo_camera'>
-    <pose>0 0 0 0 0 0</pose>
-    <inertial>
+      <mass value="5.0"/>
+      <geometry>
+        <cylinder length="0.05" radius="0.1"/>
+      </geometry>
+    </collision>
+  </link>
+  <!--Joints to chassis-->
+	<joint type="continuous" name="left_wheel_hinge">
+	  <origin xyz="0 -0.2 -0.05" rpy="0 0 0"/>
+	  <child link="left_drive_wheel"/>
+	  <parent link="chassis"/>
+	  <axis xyz="0 1 0" rpy="0 0 0"/>
+	  <limit effort="10000" velocity="1000"/>
+	  <dynamics damping="1.0" friction="1.0"/>
+	</joint>
+	<joint type="continuous" name="right_wheel_hinge">
+	  <origin xyz="0 0.2 -0.05" rpy="0 0 0"/>
+	  <child link="right_drive_wheel"/>
+	  <parent link="chassis"/>
+	  <axis xyz="0 1 0" rpy="0 0 0"/>
+	  <limit effort="10000" velocity="1000"/>
+	  <dynamics damping="1.0" friction="1.0"/>
+	</joint>
+  <!--Front Camera-->
+  <link name="camera">
+  	<inertial>
       <mass value="0.1"/>
-      <origin xyz="0.0 0 0" rpy="0.0 0 0"/>
+      <origin xyz="0 0 0" rpy=" 0 0 0"/>
       <inertia
           ixx="1e-6" ixy="0" ixz="0"
@@ -134,27 +167,26 @@
       <origin xyz="0 0 0" rpy=" 0 0 0"/>
       <geometry>
-        <box size="0.05 0.1 0.05"/>
-      </geometry>
+  		<box size=".05 .1 .05"/>
+  	  </geometry>
     </collision>
     <visual name='camera_visual'>
-      <origin xyz="0 0 0" rpy="0 0 0"/>
-      <geometry>
-        <box size="0.05 0.05 0.05"/>
-      </geometry>
-    </visual>
-  </link>
-  <joint type="fixed" name="camera_joint">
-    <origin xyz="0.2 0 0" rpy="0 0 0"/>
-    <child link="stereo_camera"/>
-    <parent link="chassis"/>
-    <axis xyz="0 1 0" rpy="0 0 0"/>
-    <limit effort="10000" velocity="1000"/>
-    <dynamics damping="1.0" friction="1.0"/>
+      <origin xyz="0.0 0 0" rpy=" 0 0 0"/>
+      <geometry>
+  		<box size=".05 .1 .05"/>
+  	  </geometry>
+    </visual>
+  </link>
+  <!--Camera Joint-->
+  <joint name="camera_joint" type="fixed">
+  	<origin xyz="0.35 0 0" rpy="0 0 0" />
+  	<parent link="chassis" />
+  	<child link="camera" />
+  	<axis xyz="0 1 0" rpy="0 0 0" />
   </joint>
-  <link name='hokuyo_lidar'>
-    <pose>0 0 0 0 0 0</pose>
-    <inertial>
+  <!--Lidar-->
+  <link name="hokuyo">
+  	<inertial>
       <mass value="1e-5"/>
-      <origin xyz="0.0 0 0" rpy="0.0 0 0"/>
+      <origin xyz="0.0 0 0" rpy=" 0 0 0"/>
       <inertia
           ixx="1e-6" ixy="0" ixz="0"
@@ -163,24 +195,23 @@
       />
     </inertial>
-    <collision name='lidar_collision'>
-      <origin xyz="0 0 0" rpy=" 0 0 0"/>
-      <geometry>
-        <box size="0.1 0.1 0.1"/>
-      </geometry>
-    </collision>
-    <visual name='lidar_visual'>
-      <origin xyz="0 0 0" rpy="0 0 0"/>
-      <geometry>
-        <mesh filename="package://my_robot/meshes/hokuyo.dae"/>
-      </geometry>
-    </visual>
-  </link>
-  <joint type="fixed" name="lidar_joint">
-    <origin xyz="0.15 0.0 0.1" rpy="0 0 0"/>
-    <child link="hokuyo_lidar"/>
-    <parent link="chassis"/>
-    <axis xyz="0 1 0" rpy="0 0 0"/>
-    <limit effort="10000" velocity="1000"/>
-    <dynamics damping="1.0" friction="1.0"/>
+    <collision name='hokuyo_collision'>
+      <origin xyz="0 0 0" rpy=" 0 0 0"/>
+      <geometry>
+  		<box size="0.1 0.1 0.1"/>
+  	  </geometry>
+    </collision>
+    <visual name='hokuyo_visual'>
+      <origin xyz="0 0 0" rpy=" 0 0 0"/>
+      <geometry>
+  		<mesh filename="package://my_robot/meshes/hokuyo.dae" />
+  	  </geometry>
+    </visual>
+  </link>
+  <!--LidarJoint-->
+  <joint name="hokuyo_joint" type="fixed">
+  	<origin xyz="0.3 0 0.1" rpy="0 0 0" />
+  	<parent link="chassis" />
+  	<child link="hokuyo" />
+  	<axis xyz="0 1 0" rpy="0 0 0" />
   </joint>
 </robot>
